Commit message: working code

File: cart_pole_3d_description/urdf/cart_pole_3d.urdf (robot description, URDF)
Before this commit: robot cart_pole_3d, 3 links, 2 joints
Links:
- added link world
Joints:
- added joint fixed: type fixed, parent world, child base_link
- joint base_cart_joint: limit lower=-0.75 upper=0.75 effort=10000 velocity=2 -> lower=-2 upper=2 effort=2000000 velocity=100000
- joint cart_pole_joint: limit lower=-0.5 upper=0.5 effort=0 velocity=0 -> lower=-1 upper=1 effort=1 velocity=100
